Commit message: automatic sim2real joints matching based on fixed URDF joints

File: nico_upper_rh6d_r.urdf (robot description, URDF)
Before this commit: robot nico_upper_rh6d, 20 links, 19 joints
Joints:
- removed joint r_wrist_z_rjoint
- added joint r_wrist_z: type revolute, parent right_lower_arm, child right_wrist, origin xyz=0 0 -0.105 rpy=0 0 1.57, axis 0 0 1, limit lower=1.46608 upper=1.67552 effort=30 velocity=1

Commit message: automatic execution cotrol, body update, execution error logging

File: nico_upper_rh6d_r.urdf (robot description, URDF)
Before this commit: robot nico_upper_rh6d, 20 links, 19 joints
Links:
- link endeffectol: mass None -> 0.000009
- link endeffector: mass None -> 0.000009
- link torso: mass None -> 0.090439

Commit message: old solver bugfix - verbobse added, urdf wrist limits updted, angle error corrected - wrist angle WIP

File: nico_upper_rh6d_r.urdf (robot description, URDF)
Before this commit: robot nico_upper_rh6d, 20 links, 19 joints
Joints:
- joint r_wrist_x: limit lower=-0.785398 upper=0 effort=30 velocity=1 -> lower=-0.872664626 upper=0.52 effort=30 velocity=1
- joint r_wrist_z: limit lower=1.46608 upper=1.67552 effort=30 velocity=1 -> lower=-1.5707963268 upper=1.5707963268 effort=30 velocity=1

Commit message: urdf updated, hnd angles rescaled, nicorad2deg WIP

File: nico_upper_rh6d_r.urdf (robot description, URDF)
Before this commit: robot nico_upper_rh6d, 20 links, 19 joints
Joints:
- joint r_wrist_x: axis 0 1 0 -> 0 -1 0

Commit message: Ik solver bugfix

File: nico_upper_rh6d_r.urdf (robot description, URDF)
Before this commit: robot nico_upper_rh6d, 20 links, 19 joints
Joints:
- joint r_wrist_z: limit lower=-1.5707963268 upper=1.5707963268 effort=30 velocity=1 -> lower=1.4 upper=1.57 effort=30 velocity=1

Commit message: urdf hand update angles, ik solver - finger orientation parameter added

File: nico_upper_rh6d_r.urdf (robot description, URDF)
Before this commit: robot nico_upper_rh6d, 20 links, 19 joints
Joints:
- joint r_wrist_x: limit lower=-0.872664626 upper=0.52 effort=30 velocity=1 -> lower=-0.785398163 upper=0.785398163 effort=30 velocity=1
- joint r_wrist_z: limit lower=1.4 upper=1.57 effort=30 velocity=1 -> lower=-1.57079633 upper=1.57079633 effort=30 velocity=1
